File: stm8mdbdo/_autosave-stm8do.kicad_pcb (KiCad board)
At the start: 2 copper layers, 63 parts, among them J1 Conn_01x02, P1 CONN_01X02, P2 PRG, P3 DIN, P4 AIN, P5 DO, U1 MC34063AD, U2 STM8S003F3P, U3 TLP185, U4 TLP185, U5 TLP185, U6 MAX485, Y1 Crystal

Commit message: Auto commit
Parts:
- C7: value CP_Small -> 100uF
- moved D2 80.5 mm to (106.7, 146.1)
- moved C3 3.59 mm to (123.2, 166.4)
- moved L1 1.27 mm to (104.1, 156.2), turned to 90 degrees
Changed lines of the file:
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@@
     (36 B.SilkS user)
     (37 F.SilkS user)
-    (38 B.Mask user)
-    (39 F.Mask user)
-    (40 Dwgs.User user)
-    (41 Cmts.User user)
-    (42 Eco1.User user)
-    (43 Eco2.User user)
-    (44 Edge.Cuts user)
-    (45 Margin user)
-    (46 B.CrtYd user)
+    (38 B.Mask user hide)
+    (39 F.Mask user hide)
+    (40 Dwgs.User user hide)
+    (41 Cmts.User user hide)
+    (42 Eco1.User user hide)
+    (43 Eco2.User user hide)
+    (44 Edge.Cuts user hide)
+    (45 Margin user hide)
+    (46 B.CrtYd user hide)
     (47 F.CrtYd user)
     (48 B.Fab user)
-    (49 F.Fab user)
+    (49 F.Fab user hide)
   )
   (setup
@@
   )
   (module Capacitor_THT:CP_Radial_D10.0mm_P5.00mm (layer F.Cu)
-    (at 125.73 168.91)
+    (at 123.19 166.37)
     (descr "CP, Radial series, Radial, pin pitch=5.00mm, , diameter=10mm, Electrolytic Capacitor")
     (tags "CP Radial series Radial pin pitch 5.00mm  diameter 10mm Electrolytic Capacitor")
@@
       (effects (font (size 1 1) (thickness 0.15)))
     )
-    (fp_text value CP_Small (at 2.5 6.25) (layer F.Fab)
+    (fp_text value 100uF (at 2.5 6.25) (layer F.Fab)
       (effects (font (size 1 1) (thickness 0.15)))
     )
@@
   )
   (module Diode_SMD:D_0805_2012Metric_Pad1.15x1.40mm_HandSolder (layer F.Cu)
-    (at 150.480001 78.490001)
+    (at 106.68 146.05)
     (descr "Diode SMD 0805 (2012 Metric), square (rectangular) end terminal, IPC_7351 nominal, (Body size source: https://docs.google.com/spreadsheets/d/1BsfQQcO9C6DZCsRaXUlFlo91Tg2WpOkGARC1WS5S8t0/edit?usp=sharing), generated with kicad-footprint-generator")
     (tags "diode handsolder")
@@
   )
   (module Inductor_SMD:L_2816_7142Metric_Pad3.20x4.45mm_HandSolder (layer F.Cu)
-    (at 104.14 154.94 270)
+    (at 104.14 156.21 90)
     (descr "Capacitor SMD 2816 (7142 Metric), square (rectangular) end terminal, IPC_7351 nominal with elongated pad for handsoldering. (Body size from: https://www.vishay.com/docs/30100/wsl.pdf), generated with kicad-footprint-generator")
     (tags "inductor handsolder")
     (attr smd)
-    (fp_text reference L1 (at 0 -3.18 270) (layer F.SilkS)
-      (effects (font (size 1 1) (thickness 0.15)))
-    )
-    (fp_text value 220uH (at 0 3.18 270) (layer F.Fab)
-      (effects (font (size 1 1) (thickness 0.15)))
-    )
-    (fp_text user %R (at 0 0 270) (layer F.Fab)
+    (fp_text reference L1 (at 0 -3.18 90) (layer F.SilkS)
+      (effects (font (size 1 1) (thickness 0.15)))
+    )
+    (fp_text value 220uH (at 0 3.18 90) (layer F.Fab)
+      (effects (font (size 1 1) (thickness 0.15)))
+    )
+    (fp_text user %R (at 0 0 90) (layer F.Fab)
       (effects (font (size 1 1) (thickness 0.15)))
     )
@@
     (fp_line (start -3.55 -2.1) (end 3.55 -2.1) (layer F.Fab) (width 0.1))
     (fp_line (start -3.55 2.1) (end -3.55 -2.1) (layer F.Fab) (width 0.1))
-    (pad 2 smd roundrect (at 2.6 0 270) (size 3.2 4.45) (layers F.Cu F.Paste F.Mask) (roundrect_rratio 0.078125)
+    (pad 2 smd roundrect (at 2.6 0 90) (size 3.2 4.45) (layers F.Cu F.Paste F.Mask) (roundrect_rratio 0.078125)
       (net 8 +5V))
-    (pad 1 smd roundrect (at -2.6 0 270) (size 3.2 4.45) (layers F.Cu F.Paste F.Mask) (roundrect_rratio 0.078125)
+    (pad 1 smd roundrect (at -2.6 0 90) (size 3.2 4.45) (layers F.Cu F.Paste F.Mask) (roundrect_rratio 0.078125)
       (net 17 "Net-(D1-Pad1)"))
     (model ${KISYS3DMOD}/Inductor_SMD.3dshapes/L_2816_7142Metric.wrl
