File: stm8mdbdo/stm8do.kicad_pcb (KiCad board)
At the start: 2 copper layers, 177.8 x 114.3 mm, 32 parts, among them P5 CONN_01X05, U1 MC34063AD, U2 STM8S003F3P, U3 OPTO-TRANSISTOR-4, U4 MAX485

Commit message: Auto commit
Parts:
- added C12: 22pF, Capacitor_SMD:C_0805_2012Metric_Pad1.15x1.40mm_HandSolder, F.Cu at (190.5, 120.4)
- added C13: C_Small, Capacitor_SMD:C_0805_2012Metric_Pad1.15x1.40mm_HandSolder, F.Cu at (133.0, 102.4)
- added C14: C_Small, Capacitor_SMD:C_0805_2012Metric_Pad1.15x1.40mm_HandSolder, F.Cu at (129.2, 106.4)
- added C15: 470pF, Capacitor_SMD:C_0805_2012Metric_Pad1.15x1.40mm_HandSolder, F.Cu at (103.5, 116.9)
- added C3: 470uF, Capacitor_THT:CP_Radial_D10.0mm_P5.00mm, F.Cu at (104.6, 88.0)
- added C5: 0.1 uF, Capacitor_SMD:C_0805_2012Metric_Pad1.15x1.40mm_HandSolder, F.Cu at (203.4, 110.5)
- added C6: 470 nF, Capacitor_SMD:C_0805_2012Metric_Pad1.15x1.40mm_HandSolder, F.Cu at (200.7, 120.9)
- added C7: CP_Small, Capacitor_THT:CP_Radial_D10.0mm_P5.00mm, F.Cu at (125.1, 82.7)
- added D12: BTS4140N, Package_TO_SOT_SMD:SOT-223, F.Cu at (125.7, 91.6)
- added D13: MM3Z5V1, Diode_SMD:D_0805_2012Metric, F.Cu at (140.3, 103.5)
- added D3: LED, LED_SMD:LED_0805_2012Metric_Pad1.15x1.40mm_HandSolder, F.Cu at (129.2, 102.4)
- added D4: LED, LED_SMD:LED_0805_2012Metric_Pad1.15x1.40mm_HandSolder, F.Cu at (150.5, 80.5)
- added D5: LED, LED_SMD:LED_0805_2012Metric_Pad1.15x1.40mm_HandSolder, F.Cu at (142.2, 89.9)
- added D6: LED, LED_SMD:LED_0805_2012Metric_Pad1.15x1.40mm_HandSolder, F.Cu at (135.8, 93.7)
- added D7: LED, LED_SMD:LED_0805_2012Metric_Pad1.15x1.40mm_HandSolder, F.Cu at (132.0, 93.5)
- added J1: Conn_01x02, Connector_PinHeader_1.27mm:PinHeader_1x02_P1.27mm_Vertical, F.Cu at (114.4, 115.5)
- added P1: CONN_01X02, Connector_PinHeader_1.27mm:PinHeader_1x02_P1.27mm_Vertical_SMD_Pin1Left, F.Cu at (133.6, 90.7)
- added P2: CONN_01X04, Connector_PinHeader_1.27mm:PinHeader_1x04_P1.27mm_Horizontal, F.Cu at (121.3, 100.7)
- added P3: CONN_01X04, Connector_PinHeader_1.27mm:PinHeader_1x04_P1.27mm_Horizontal, F.Cu at (131.1, 96.4)
- added P4: CONN_01X02, Connector_PinHeader_1.27mm:PinHeader_1x02_P1.27mm_Vertical_SMD_Pin1Left, F.Cu at (144.3, 86.7)
- added R1: 0.33, Resistor_SMD:R_0805_2012Metric_Pad1.15x1.40mm_HandSolder, F.Cu at (139.0, 95.7)
- added R14: R, Resistor_SMD:R_0805_2012Metric_Pad1.15x1.40mm_HandSolder, F.Cu at (149.7, 87.8)
- added R15: 120, Resistor_SMD:R_0805_2012Metric_Pad1.15x1.40mm_HandSolder, F.Cu at (114.7, 113.4)
- added R16: 20K, Resistor_SMD:R_0805_2012Metric_Pad1.15x1.40mm_HandSolder, F.Cu at (111.0, 116.9)
- added R17: 20K, Resistor_SMD:R_0805_2012Metric_Pad1.15x1.40mm_HandSolder, F.Cu at (114.7, 111.4)
- added R18: 20K, Resistor_SMD:R_0805_2012Metric_Pad1.15x1.40mm_HandSolder, F.Cu at (111.0, 113.4)
- added R19: 20K, Resistor_SMD:R_0805_2012Metric_Pad1.15x1.40mm_HandSolder, F.Cu at (107.2, 116.9)
- added R20: 20K, Resistor_SMD:R_0805_2012Metric_Pad1.15x1.40mm_HandSolder, F.Cu at (111.0, 111.4)
- added U5: TLP185, Package_SO:SOIC-4_4.55x3.7mm_P2.54mm, F.Cu at (137.2, 79.6)
- added U6: MAX485, Package_SO:SOIC-8_3.9x4.9mm_P1.27mm, F.Cu at (105.4, 113.2)
- added Y1: Crystal, Crystal:Crystal_SMD_HC49-SD_HandSoldering, F.Cu at (195.6, 116.0)
- C1, C2, C4: footprint Capacitors_SMD:C_0805_HandSoldering -> Capacitor_SMD:C_0805_2012Metric_Pad1.15x1.40mm_HandSolder
- C10, C8, C9: value C_Small -> 470pF; footprint Capacitors_SMD:C_0805_HandSoldering -> Capacitor_SMD:C_0805_2012Metric_Pad1.15x1.40mm_HandSolder
- C11: value C_Small -> 22pF; footprint Capacitors_SMD:C_0805_HandSoldering -> Capacitor_SMD:C_0805_2012Metric_Pad1.15x1.40mm_HandSolder
- D1: footprint Diodes_SMD:DO-214AB_Handsoldering -> Diode_SMD:D_SMC
- D10, D11, D9: footprint TO_SOT_Packages_SMD:SOT-223 -> Package_TO_SOT_SMD:SOT-223
- D2: value D -> MM3Z5V1; footprint Diodes_SMD:D_0805 -> Diode_SMD:D_0805_2012Metric_Pad1.15x1.40mm_HandSolder
- D8: value BTS4140N -> MM3Z5V1; footprint TO_SOT_Packages_SMD:SOT-223 -> Diode_SMD:D_0805_2012Metric
- L1: value INDUCTOR -> 220uH; footprint Inductors:Inductor_Taiyo-Yuden_NR-80xx_HandSoldering -> Inductor_SMD:L_2816_7142Metric_Pad3.20x4.45mm_HandSolder
- P5: footprint Connectors_Phoenix:PhoenixContact_MSTBV-GF_05x5.08mm_Vertical_ThreadedFlange -> Connector_PinHeader_1.27mm:PinHeader_1x05_P1.27mm_Vertical_SMD_Pin1Left
- R10: value R -> 10K; footprint Resistors_SMD:R_0805_HandSoldering -> Resistor_SMD:R_0805_2012Metric_Pad1.15x1.40mm_HandSolder
- R11, R12, R13, R2, R3, R4, R5, R6, R8, R9: footprint Resistors_SMD:R_0805_HandSoldering -> Resistor_SMD:R_0805_2012Metric_Pad1.15x1.40mm_HandSolder
- R7: value 10K -> 1.2k; footprint Resistors_SMD:R_0805_HandSoldering -> Resistor_SMD:R_0805_2012Metric_Pad1.15x1.40mm_HandSolder
- RN1: value R_Pack05 -> R_Pack04; footprint Resistors_SMD:R_Array_Convex_5x1206 -> Resistor_SMD:R_Array_Concave_4x0603
- U1: footprint Housings_SOIC:SOIC-8_3.9x4.9mm_Pitch1.27mm -> Package_SO:SOIC-8_3.9x4.9mm_P1.27mm
- U2: footprint Housings_SSOP:TSSOP-20_4.4x6.5mm_Pitch0.65mm -> Package_SO:TSSOP-20_4.4x6.5mm_P0.65mm
- U3: value OPTO-TRANSISTOR-4 -> TLP185; footprint Opto-Devices:Optocoupler_SMD_ReflowWaveSoldering_KPC357_LTV35x_PC357_SingleChannel -> Package_SO:SOIC-4_4.55x3.7mm_P2.54mm
- U4: value MAX485 -> TLP185; footprint Housings_SOIC:SOIC-8_3.9x4.9mm_Pitch1.27mm -> Package_SO:SOIC-4_4.55x3.7mm_P2.54mm
- moved D11 103.2 mm to (116.8, 93.6)
- moved U2 97.8 mm to (207.9, 116.0)
- moved D9 97.3 mm to (116.8, 86.3)
- moved C4 95.9 mm to (136.7, 106.3)
- moved C8 93.1 mm to (146.5, 97.3)
- moved R4 89.0 mm to (136.7, 104.3)
- moved C1 88.1 mm to (139.6, 93.6)
- moved R9 80.0 mm to (150.4, 82.5)
- moved C10 77.9 mm to (139.0, 97.6)
- moved C2 77.7 mm to (149.7, 91.7), turned to 0 degrees
- moved P5 76.0 mm to (145.0, 81.2), turned to 0 degrees
- moved C9 74.4 mm to (142.7, 95.6)
- moved D2 70.6 mm to (150.5, 78.5)
- moved R11 69.6 mm to (143.3, 93.4)
- moved U3 69.3 mm to (125.6, 97.4)
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Connections:
- C10 pad 1: AIN1 -> /EXT_GND
- C10 pad 2: GND -> Net-(C10-Pad2)
- C11 pad 1: AIN2 -> GND
- C11 pad 2: GND -> Net-(C11-Pad2)
- C8 pad 1: GND -> /EXT_GND
- C9 pad 1: GND -> /EXT_GND
- D10 pad 1: OUT3 -> OUT2
- D11 pad 1: OUT4 -> OUT3
- D8 pad 1: OUT1 -> AIN1
- D8 pad 2: Vbb -> GND
- D9 pad 1: OUT2 -> OUT1
- P5 pad 2: Net-(D8-Pad3) -> Net-(D9-Pad3)
- P5 pad 3: Net-(D9-Pad3) -> Net-(D10-Pad3)
- P5 pad 4: Net-(D10-Pad3) -> Net-(D11-Pad3)
- R10 pad 1: Net-(P4-Pad1) -> +5V
- R10 pad 2: AIN1 -> IN3
- R11 pad 1: GND -> Net-(P4-Pad1)
- R12 pad 1: AIN2 -> GND
- R12 pad 2: Net-(P4-Pad2) -> AIN1
- R13 pad 1: GND -> AIN2
- R13 pad 2: AIN2 -> Net-(P4-Pad2)
- R4 pad 1: Net-(R4-Pad1) -> Net-(C9-Pad2)
- R5 pad 1: Net-(R5-Pad1) -> Net-(C8-Pad2)
- R6 pad 2: Net-(R6-Pad2) -> Net-(C10-Pad2)
- R7 pad 1: +5V -> Net-(D3-Pad2)
- R7 pad 2: IN1 -> STATUS
- R8 pad 2: IN2 -> IN1
- R9 pad 2: IN3 -> IN2
- RN1 pad 1: STATUS -> Net-(D7-Pad2)
- RN1 pad 2: OUT1 -> Net-(D6-Pad2)
- RN1 pad 3: OUT2 -> Net-(D5-Pad2)
- RN1 pad 4: OUT3 -> Net-(D4-Pad2)
- RN1 pad 5: OUT4 -> OUT1
- RN1 pad 6: Net-(D7-Pad2) -> OUT2
- RN1 pad 7: Net-(D6-Pad2) -> OUT3
- RN1 pad 8: Net-(D5-Pad2) -> OUT4
- U2 pad 5: Net-(C8-Pad2) -> Net-(C11-Pad2)
- U2 pad 6: Net-(C9-Pad2) -> Net-(C12-Pad2)
- U3 pad 1: Net-(R4-Pad1) -> Net-(C8-Pad2)
- U3 pad 3: Net-(R5-Pad1) -> /EXT_GND
- U3 pad 4: Net-(P3-Pad1) -> GND
- U4 pad 1: RO -> Net-(C9-Pad2)
- U4 pad 3: IN/OUT -> /EXT_GND
- U4 pad 4: DI -> GND
- U4 pad 6: A -> IN2
Other:
- board outline removed
- net class Default: via_dia 0.6 -> 0.8
- rule pad_to_mask_clearance: 0.2 -> 0

Commit message: Auto commit
Parts:
- C4: value C_Small -> 470pF
- C7: value CP_Small -> 100uF
- P2: value CONN_01X04 -> PRG; footprint Connector_PinHeader_1.27mm:PinHeader_1x04_P1.27mm_Horizontal -> Connector_PinHeader_1.27mm:PinHeader_1x04_P1.27mm_Vertical
- P3: value CONN_01X04 -> DIN
- P4: value CONN_01X02 -> AIN
- P5: value CONN_01X05 -> DO
- moved L1 105.3 mm to (104.1, 156.2), turned to 90 degrees
- moved P2 85.9 mm to (207.0, 105.4), turned to 90 degrees
- moved C3 80.5 mm to (123.2, 166.4)
- moved D2 80.5 mm to (106.7, 146.1)
- moved R2 72.5 mm to (132.1, 156.2), turned to 180 degrees
- moved R3 65.3 mm to (137.2, 156.2)
- moved D1 59.2 mm to (116.8, 154.9), turned to 270 degrees
- moved C7 59.0 mm to (115.6, 141.0)
- moved U1 49.8 mm to (130.8, 151.1)
- moved R1 49.8 mm to (130.8, 144.8)
- moved C4 49.2 mm to (124.5, 153.9), turned to 270 degrees

Commit message: Auto commit
Parts:
- P5: footprint Connector_PinHeader_1.27mm:PinHeader_1x05_P1.27mm_Vertical_SMD_Pin1Left -> Connector_PinHeader_1.27mm:PinHeader_1x05_P1.27mm_Vertical
- moved D10 148.1 mm to (254.0, 97.8), turned to 180 degrees
- moved D11 138.7 mm to (254.6, 109.2), turned to 180 degrees
- moved D9 137.8 mm to (254.6, 87.6), turned to 180 degrees
- moved D12 131.6 mm to (254.0, 120.7), turned to 180 degrees
- moved P5 128.2 mm to (271.8, 100.3)
- moved U5 66.9 mm to (195.6, 47.0)

Commit message: Auto commit
Parts:
- added J2: Screw_Terminal_01x02, TerminalBlock:TerminalBlock_bornier-2_P5.08mm, F.Cu at (103.5, 136.0)
- P1: footprint Connector_PinHeader_1.27mm:PinHeader_1x02_P1.27mm_Vertical_SMD_Pin1Left -> TerminalBlock:TerminalBlock_bornier-2_P5.08mm
- P2: footprint Connector_PinHeader_1.27mm:PinHeader_1x04_P1.27mm_Vertical -> Connector_Wire:SolderWirePad_1x04_P3.81mm_Drill1.2mm
- P3: footprint Connector_PinHeader_1.27mm:PinHeader_1x04_P1.27mm_Horizontal -> TerminalBlock:TerminalBlock_bornier-4_P5.08mm
- P4: footprint Connector_PinHeader_1.27mm:PinHeader_1x02_P1.27mm_Vertical_SMD_Pin1Left -> TerminalBlock:TerminalBlock_bornier-3_P5.08mm
- P5: footprint Connector_PinHeader_1.27mm:PinHeader_1x05_P1.27mm_Vertical -> TerminalBlock:TerminalBlock_bornier-6_P5.08mm
- moved P5 173.2 mm to (103.5, 59.5)
- moved D9 156.5 mm to (99.1, 70.0), turned to 270 degrees
- moved D10 147.4 mm to (109.3, 70.0), turned to 270 degrees
- moved D11 139.5 mm to (120.7, 70.0), turned to 270 degrees
- moved D12 132.0 mm to (132.2, 70.0), turned to 270 degrees
- moved U5 123.9 mm to (74.0, 71.0), turned to 270 degrees
- moved U2 87.7 mm to (122.7, 95.3), turned to 90 degrees
- moved C5 86.9 mm to (117.2, 99.7), turned to 270 degrees
- moved D8 82.8 mm to (72.9, 123.5)
- moved P4 82.2 mm to (78.5, 136.0)
- moved R11 78.1 mm to (73.0, 127.5), turned to 180 degrees
- moved R14 77.7 mm to (79.0, 120.0)
- moved R6 76.1 mm to (74.0, 65.0)
- moved C6 75.3 mm to (127.6, 102.5), turned to 180 degrees
- moved Y1 73.3 mm to (122.7, 107.6), turned to 0 degrees
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Routing:
- net +5V: track 0.00 -> 139.8 mm, vias 0 -> 2
- net Vbb: track 0.00 -> 66.1 mm, vias 0 -> 4
- net GND: track 0.00 -> 51.4 mm, vias 0 -> 14
- net OUT4: track 0.00 -> 46.5 mm
- net /EXT_GND: track 0.00 -> 43.1 mm
- net OUT2: track 0.00 -> 39.3 mm, vias 0 -> 2
- net OUT3: track 0.00 -> 38.7 mm, vias 0 -> 2
- net Net-(D1-Pad1): track 0.00 -> 35.4 mm
- net Net-(C3-Pad1): track 0.00 -> 34.2 mm
- net OUT1: track 0.00 -> 30.7 mm
- net AIN1: track 0.00 -> 20.6 mm
- net AIN2: track 0.00 -> 19.8 mm
- net Net-(D7-Pad2): track 0.00 -> 18.9 mm
- net Net-(C12-Pad2): track 0.00 -> 18.4 mm
- net Net-(C11-Pad2): track 0.00 -> 18.2 mm
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Other:
- board outline added: 68 x 85 mm
- net class ANALOG added: clearance 0.2, trace_width 0.4, via_dia 0.8, via_drill 0.4
- net class LOAD_POWER added: clearance 0.2, trace_width 0.8, via_dia 1, via_drill 0.6
- net class POWER added: clearance 0.2, trace_width 0.8, via_dia 0.8, via_drill 0.4
- board text added: "+12/24V"
- board text added: "+5V"
- board text added: "."
- board text added: "GND"
- board text added: "NRST"
- board text added: "SWIM"
- board text added: "TERM"

Commit message: Auto commit
Parts:
- C1, C2: moved to B.Cu
- moved C2 11.8 mm to (120.5, 100.5), turned to 180 degrees
- moved C1 8.95 mm to (120.5, 98.5), turned to 180 degrees
- moved P1 5.00 mm to (129.0, 136.0), turned to 180 degrees
Connections:
- net A renamed A+
- net B renamed B-
- C1 pad 1: Net-(C1-Pad1) -> +5V
- C1 pad 2: Net-(C1-Pad2) -> GND
- C2 pad 1: Net-(C1-Pad1) -> +5V
- C2 pad 2: Net-(C1-Pad2) -> GND
Routing:
- net +5V: track 139.8 -> 214.0 mm, vias 2 -> 3
- net IN3: track 4.73 -> 68.5 mm, vias 0 -> 2
- net A+: track 15.0 -> 76.1 mm, vias 0 -> 1
- net IN2: track 3.85 -> 59.4 mm, vias 0 -> 2
- net AIN1: track 20.6 -> 74.0 mm
- net AIN2: track 19.8 -> 70.2 mm, vias 0 -> 2
- net STATUS: track 0.00 -> 49.7 mm, vias 0 -> 2
- net B-: track 12.7 -> 61.9 mm, vias 0 -> 1
- net IN1: track 3.76 -> 52.1 mm, vias 0 -> 2
- net IN/OUT: track 6.00 -> 52.0 mm, vias 0 -> 2
- net DI: track 5.01 -> 49.7 mm, vias 0 -> 2
- net RO: track 5.69 -> 46.7 mm, vias 0 -> 2
- net Net-(D4-Pad2): track 0.00 -> 22.5 mm, vias 0 -> 2
- net Net-(C9-Pad2): track 2.85 -> 16.7 mm, vias 0 -> 2
- net GND: track 51.4 -> 64.9 mm, vias 14 -> 20
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- added copper zone on B.Cu, net GND
Other:
- board text added: "A+"
- board text added: "AIN1"
- board text added: "AIN2"
- board text added: "B-"
- board text added: "CP"
- board text added: "DO1"
- board text added: "DO2"
- board text added: "DO3"
- board text added: "DO4"
- board text added: "NC"
- board text added: "POWER"

Commit message: Auto commit
Parts:
- D1: footprint Diode_SMD:D_SMC -> Diode_SMD:D_SMA
- J1: footprint Connector_PinHeader_1.27mm:PinHeader_1x02_P1.27mm_Vertical -> Connector_PinHeader_2.54mm:PinHeader_1x02_P2.54mm_Vertical
- Y1: footprint Crystal:Crystal_SMD_HC49-SD_HandSoldering -> Crystal:Crystal_SMD_HC49-SD
Routing:
- net Net-(D1-Pad1): track 38.1 -> 39.5 mm
- net GND: track 64.9 -> 66.3 mm, vias 20 -> 23
- net A+: track 76.1 -> 76.6 mm
- added copper zone on F.Cu, net GND
Other:
- board text added: "IN1"
- board text added: "IN2"
- board text added: "IN3"

Commit message: Auto commit
Parts:
- moved D5 1.83 mm to (110.6, 80.3)
- moved D6 0.88 mm to (121.3, 80.3)
Routing:
- net Net-(D5-Pad2): track 10.7 -> 8.82 mm
- net Net-(D6-Pad2): track 8.90 -> 9.78 mm
Changed lines of the file:
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@@
   (general
     (thickness 1.6)
-    (drawings 37)
-    (tracks 629)
+    (drawings 38)
+    (tracks 628)
     (zones 0)
     (modules 64)
@@
     (32 B.Adhes user hide)
     (33 F.Adhes user hide)
-    (34 B.Paste user hide)
-    (35 F.Paste user hide)
-    (36 B.SilkS user hide)
+    (34 B.Paste user)
+    (35 F.Paste user)
+    (36 B.SilkS user)
     (37 F.SilkS user)
     (38 B.Mask user hide)
@@
     (42 Eco1.User user hide)
     (43 Eco2.User user hide)
-    (44 Edge.Cuts user hide)
+    (44 Edge.Cuts user)
     (45 Margin user hide)
     (46 B.CrtYd user hide)
@@
     (visible_elements 7FFFFFFF)
     (pcbplotparams
-      (layerselection 0x010fc_ffffffff)
-      (usegerberextensions false)
+      (layerselection 0x010f0_ffffffff)
+      (usegerberextensions true)
       (usegerberattributes false)
       (usegerberadvancedattributes false)
       (creategerberjobfile false)
-      (excludeedgelayer true)
+      (excludeedgelayer false)
       (linewidth 0.100000)
       (plotframeref false)
@@
       (plotvalue true)
       (plotinvisibletext false)
-      (padsonsilk false)
+      (padsonsilk true)
       (subtractmaskfromsilk false)
       (outputformat 1)
       (mirror false)
-      (drillshape 1)
+      (drillshape 0)
       (scaleselection 1)
-      (outputdirectory ""))
+      (outputdirectory "GERBER/"))
   )
   (net 0 "")
@@
   )
   (module LED_SMD:LED_0805_2012Metric_Pad1.15x1.40mm_HandSolder (layer F.Cu)
-    (at 108.72612 80.26044 90)
+    (at 110.551533 80.26044 90)
     (descr "LED SMD 0805 (2012 Metric), square (rectangular) end terminal, IPC_7351 nominal, (Body size source: https://docs.google.com/spreadsheets/d/1BsfQQcO9C6DZCsRaXUlFlo91Tg2WpOkGARC1WS5S8t0/edit?usp=sharing), generated with kicad-footprint-generator")
     (tags "LED handsolder")
@@
   )
   (module LED_SMD:LED_0805_2012Metric_Pad1.15x1.40mm_HandSolder (layer F.Cu)
-    (at 120.39996 80.26044 90)
+    (at 121.282186 80.26044 90)
     (descr "LED SMD 0805 (2012 Metric), square (rectangular) end terminal, IPC_7351 nominal, (Body size source: https://docs.google.com/spreadsheets/d/1BsfQQcO9C6DZCsRaXUlFlo91Tg2WpOkGARC1WS5S8t0/edit?usp=sharing), generated with kicad-footprint-generator")
     (tags "LED handsolder")
@@
     (tags "SOIC SO")
     (attr smd)
-    (fp_text reference U4 (at 0 -2.8 270) (layer F.SilkS)
+    (fp_text reference U4 (at -1 -2.8 270) (layer F.SilkS)
       (effects (font (size 1 1) (thickness 0.15)))
     )
@@
     (tags "SOIC SO")
     (attr smd)
-    (fp_text reference U5 (at 0 -2.8 270) (layer F.SilkS)
+    (fp_text reference U5 (at -0.5 3 270) (layer F.SilkS)
       (effects (font (size 1 1) (thickness 0.15)))
     )
@@
     )
   )
+  (gr_text . (at 119 99) (layer F.SilkS)
+    (effects (font (size 1.5 1.5) (thickness 0.3)))
+  )
   (gr_text IN3 (at 93.5 64.5 90) (layer B.SilkS)
     (effects (font (size 1.5 1.5) (thickness 0.3)) (justify mirror))
@@
   (segment (start 109.333902 127.573959) (end 110.786782 127.573959) (width 0.25) (layer F.Cu) (net 1))
   (segment (start 108.272182 126.705279) (end 109.333902 127.573959) (width 0.25) (layer F.Cu) (net 1))
-  (via (at 122.41672 81.3284) (size 0.8) (drill 0.4) (layers F.Cu B.Cu) (net 1))
+  (via (at 123 80.5) (size 0.8) (drill 0.4) (layers F.Cu B.Cu) (net 1))
   (segment (start 120.39996 81.28544) (end 122.37376 81.28544) (width 0.25) (layer F.Cu) (net 1))
   (segment (start 122.37376 81.28544) (end 122.41672 81.3284) (width 0.25) (layer F.Cu) (net 1))
-  (via (at 110.60572 81.3792) (size 0.8) (drill 0.4) (layers F.Cu B.Cu) (net 1))
+  (via (at 112.5 82.5) (size 0.8) (drill 0.4) (layers F.Cu B.Cu) (net 1))
   (segment (start 108.72612 81.28544) (end 110.51196 81.28544) (width 0.25) (layer F.Cu) (net 1))
   (segment (start 110.51196 81.28544) (end 110.60572 81.3792) (width 0.25) (layer F.Cu) (net 1))
@@
   (segment (start 71 69) (end 71 67.75) (width 0.25) (layer F.Cu) (net 8))
   (segment (start 71 67.75) (end 71 63.75) (width 0.25) (layer F.Cu) (net 8))
-  (segment (start 78.25 70.025) (end 78.25 69.75) (width 0.25) (layer F.Cu) (net 8))
-  (segment (start 78 70.275) (end 78.25 70.025) (width 0.25) (layer F.Cu) (net 8))
-  (segment (start 78 70.95) (end 78 70.275) (width 0.25) (layer F.Cu) (net 8))
   (segment (start 79.75 69.75) (end 78.25 69.75) (width 0.25) (layer F.Cu) (net 8))
-  (segment (start 78.25 69.75) (end 71.75 69.75) (width 0.25) (layer F.Cu) (net 8))
-  (segment (start 78 69.5) (end 78.25 69.75) (width 0.25) (layer F.Cu) (net 8))
-  (segment (start 78 68.05) (end 78 69.5) (width 0.25) (layer F.Cu) (net 8))
   (segment (start 86.5 71.7) (end 86.5 69.75) (width 0.25) (layer F.Cu) (net 8))
   (segment (start 88 69.75) (end 86.5 69.75) (width 0.25) (layer F.Cu) (net 8))
   (segment (start 86.5 69.75) (end 79.75 69.75) (width 0.25) (layer F.Cu) (net 8))
+  (segment (start 78.25 69.75) (end 78 69.75) (width 0.25) (layer F.Cu) (net 8))
+  (segment (start 78 69.75) (end 71.75 69.75) (width 0.25) (layer F.Cu) (net 8))
+  (segment (start 78 68.05) (end 78 70) (width 0.25) (layer F.Cu) (net 8))
+  (segment (start 78 70.95) (end 78 70) (width 0.25) (layer F.Cu) (net 8))
+  (segment (start 78 70) (end 78 69.75) (width 0.25) (layer F.Cu) (net 8))
   (segment (start 83.025 67.505) (end 83.27 67.75) (width 0.25) (layer F.Cu) (net 9))
   (segment (start 83.025 65) (end 83.025 67.505) (width 0.25) (layer F.Cu) (net 9))
@@
   (segment (start 99.75 79.16456) (end 99.82088 79.23544) (width 0.25) (layer F.Cu) (net 17))
   (segment (start 99.75 77.5) (end 99.75 79.16456) (width 0.25) (layer F.Cu) (net 17))
-  (segment (start 111.44392 79.23544) (end 108.72612 79.23544) (width 0.25) (layer F.Cu) (net 18))
+  (segment (start 111.44392 79.23544) (end 110.551533 79.23544) (width 0.25) (layer F.Cu) (net 18))
   (segment (start 114.92504 85.72604) (end 114.92504 82.71656) (width 0.25) (layer F.Cu) (net 18))
   (segment (start 114.92504 82.71656) (end 111.44392 79.23544) (width 0.25) (layer F.Cu) (net 18))
   (segment (start 115.72504 85.02604) (end 115.72504 85.72604) (width 0.25) (layer F.Cu) (net 19))
   (segment (start 115.72504 83.11036) (end 115.72504 85.02604) (width 0.25) (layer F.Cu) (net 19))
+  (segment (start 121.282186 79.23544) (end 119.59996 79.23544) (width 0.25) (layer F.Cu) (net 19))
   (segment (start 119.59996 79.23544) (end 115.72504 83.11036) (width 0.25) (layer F.Cu) (net 19))
-  (segment (start 120.39996 79.23544) (end 119.59996 79.23544) (width 0.25) (layer F.Cu) (net 19))
   (segment (start 132.01284 79.23544) (end 126.47564 79.23544) (width 0.25) (layer F.Cu) (net 20))
   (segment (start 126.47564 79.23544) (end 121.9646 83.74648) (width 0.25) (layer F.Cu) (net 20))

Commit message: Auto commit
Routing:
- net GND: vias 23 -> 20
Changed lines of the file:
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@@
     (thickness 1.6)
     (drawings 38)
-    (tracks 628)
+    (tracks 625)
     (zones 0)
     (modules 64)
@@
   (segment (start 113 99) (end 114.5 100.5) (width 0.25) (layer F.Cu) (net 1))
   (segment (start 102 123.1) (end 102 119) (width 0.8) (layer F.Cu) (net 1))
-  (via (at 72.5 101) (size 0.8) (drill 0.4) (layers F.Cu B.Cu) (net 1))
-  (via (at 75.5 105) (size 0.8) (drill 0.4) (layers F.Cu B.Cu) (net 1))
-  (via (at 72 107.5) (size 0.8) (drill 0.4) (layers F.Cu B.Cu) (net 1))
   (segment (start 118.975742 117.972759) (end 116.872622 117.972759) (width 0.6) (layer F.Cu) (net 2))
   (segment (start 119.737742 117.972759) (end 118.975742 117.972759) (width 0.6) (layer F.Cu) (net 2))
