File: stm8mdbdo/stm8do.kicad_pcb (KiCad board)
At the start: 2 copper layers, 68 x 85 mm, 64 parts, among them J1 Conn_01x02, J2 Screw_Terminal_01x02, P1 CONN_01X02, P2 PRG, P3 DIN, P4 AIN, P5 DO, U1 MC34063AD, U2 STM8S003F3P, U3 TLP185, U4 TLP185, U5 TLP185, U6 MAX485, Y1 Crystal

Commit message: Added some chems
Parts:
- added R21: 1.2k, Resistor_SMD:R_0805_2012Metric_Pad1.15x1.40mm_HandSolder, F.Cu at (103.1, 80.2)
- added R22: 1.2k, Resistor_SMD:R_0805_2012Metric_Pad1.15x1.40mm_HandSolder, F.Cu at (96.7, 80.3)
- added R23: 1.2k, Resistor_SMD:R_0805_2012Metric_Pad1.15x1.40mm_HandSolder, F.Cu at (66.2, 93.4)
- added R24: 1.2k, Resistor_SMD:R_0805_2012Metric_Pad1.15x1.40mm_HandSolder, F.Cu at (62.4, 95.4)
- added R25: 1.2k, Resistor_SMD:R_0805_2012Metric_Pad1.15x1.40mm_HandSolder, F.Cu at (66.2, 91.5)
- added R26: 1.2k, Resistor_SMD:R_0805_2012Metric_Pad1.15x1.40mm_HandSolder, F.Cu at (62.4, 93.4)
- added R27: 1.2k, Resistor_SMD:R_0805_2012Metric_Pad1.15x1.40mm_HandSolder, F.Cu at (58.7, 95.4)
- added R28: 1.2k, Resistor_SMD:R_0805_2012Metric_Pad1.15x1.40mm_HandSolder, F.Cu at (64.4, 88.1)
- D1: footprint Diode_SMD:D_SMA -> Diode_SMD:D_SMC
- J1: footprint Connector_PinHeader_2.54mm:PinHeader_1x02_P2.54mm_Vertical -> Connector_PinHeader_1.27mm:PinHeader_1x02_P1.27mm_Vertical
- P1: footprint TerminalBlock:TerminalBlock_bornier-2_P5.08mm -> Connector_PinHeader_1.27mm:PinHeader_1x02_P1.27mm_Vertical_SMD_Pin1Left
- P2: footprint Connector_Wire:SolderWirePad_1x04_P3.81mm_Drill1.2mm -> Connector_PinHeader_1.27mm:PinHeader_1x04_P1.27mm_Vertical
- P3: footprint TerminalBlock:TerminalBlock_bornier-4_P5.08mm -> Connector_PinHeader_1.27mm:PinHeader_1x04_P1.27mm_Horizontal
- P5: footprint TerminalBlock:TerminalBlock_bornier-6_P5.08mm -> Connector_PinHeader_1.27mm:PinHeader_1x05_P1.27mm_Vertical
- Y1: footprint Crystal:Crystal_SMD_HC49-SD -> Crystal:Crystal_SMD_HC49-SD_HandSoldering
Connections:
- D10 pad 1: OUT2 -> Net-(D10-Pad1)
- D11 pad 1: OUT3 -> Net-(D11-Pad1)
- D12 pad 1: OUT4 -> Net-(D12-Pad1)
- D9 pad 1: OUT1 -> Net-(D9-Pad1)
Routing:
- net Net-(R21-Pad1): track 0.00 -> 11.4 mm
- removed copper zone on B.Cu, net GND
- removed copper zone on F.Cu, net GND
Other:
- outline, holes or cut-outs redrawn
