File: stm8mdbdo/stm8do.sch (KiCad schematic (older format))
At the start: 54 parts, among them P1 CONN_01X02, P2 PRG, P3 DIN, P4 AIN, P5 DO, U1 MC34063AD, U2 STM8S003F3P, U3 TLP185, U4 TLP185, U5 TLP185, Y1 Crystal

Commit message: Auto commit
Parts:
- P4: footprint Connector_PinHeader_1.27mm:PinHeader_1x02_P1.27mm_Vertical_SMD_Pin1Left -> TerminalBlock:TerminalBlock_bornier-3_P5.08mm
Changed lines of the file:
@@
 F 0 "P4" H 10350 4900 50  0000 C CNN
 F 1 "AIN" V 10450 4750 50  0000 C CNN
-F 2 "Connector_PinHeader_1.27mm:PinHeader_1x02_P1.27mm_Vertical_SMD_Pin1Left" H 10350 4750 50  0001 C CNN
+F 2 "TerminalBlock:TerminalBlock_bornier-3_P5.08mm" H 10350 4750 50  0001 C CNN
 F 3 "" H 10350 4750 50  0000 C CNN
 	1    10350 4750

Commit message: Auto commit
Connections:
- net +5V: now also C1.1, C2.1
- net GND: now also C1.2, C2.2
Changed lines of the file:
@@
 	1250 4550 1250 4400
 Wire Wire Line
-	1250 4400 1450 4400
+	1250 4400 1350 4400
 Wire Wire Line
 	1450 4400 1450 4550
@@
 	1250 4750 1250 4900
 Wire Wire Line
-	1250 4900 1450 4900
+	1250 4900 1350 4900
 Wire Wire Line
 	1450 4900 1450 4750
@@
 L power:GND #PWR05
 U 1 1 5C687615
-P 1350 4900
-F 0 "#PWR05" H 1350 4650 50  0001 C CNN
-F 1 "GND" H 1350 4750 50  0000 C CNN
-F 2 "" H 1350 4900 50  0000 C CNN
-F 3 "" H 1350 4900 50  0000 C CNN
-	1    1350 4900
+P 1350 4950
+F 0 "#PWR05" H 1350 4700 50  0001 C CNN
+F 1 "GND" H 1350 4800 50  0000 C CNN
+F 2 "" H 1350 4950 50  0000 C CNN
+F 3 "" H 1350 4950 50  0000 C CNN
+	1    1350 4950
 	1    0    0    -1
 $EndComp
@@
 L power:+5V #PWR04
 U 1 1 5C6850AF
-P 1350 4400
-F 0 "#PWR04" H 1350 4250 50  0001 C CNN
-F 1 "+5V" H 1350 4540 50  0000 C CNN
-F 2 "" H 1350 4400 50  0000 C CNN
-F 3 "" H 1350 4400 50  0000 C CNN
-	1    1350 4400
+P 1350 4350
+F 0 "#PWR04" H 1350 4200 50  0001 C CNN
+F 1 "+5V" H 1350 4490 50  0000 C CNN
+F 2 "" H 1350 4350 50  0000 C CNN
+F 3 "" H 1350 4350 50  0000 C CNN
+	1    1350 4350
 	1    0    0    -1
 $EndComp
@@
 	0    -1   -1   0
 $EndComp
+Wire Wire Line
+	1350 4350 1350 4400
+Connection ~ 1350 4400
+Wire Wire Line
+	1350 4400 1450 4400
+Wire Wire Line
+	1350 4950 1350 4900
+Connection ~ 1350 4900
+Wire Wire Line
+	1350 4900 1450 4900
 $EndSCHEMATC

Commit message: Added some chems
Parts:
- added R21, R22, R23, R24, R25, R26, R27, R28: 1.2k, Resistor_SMD:R_0805_2012Metric_Pad1.15x1.40mm_HandSolder, symbol Device:R
Connections:
- net GND: now also R22.1, R24.1, R26.1, R28.1
- net OUT1: now also R21.2; no longer D9.1 (IN)
- net OUT2: now also R23.2; no longer D10.1 (IN)
- net OUT3: now also R25.2; no longer D11.1 (IN)
- net OUT4: now also R27.2; no longer D12.1 (IN)
- new net: R21.1, R22.2
- new net: R23.1, R24.2
- new net: R25.1, R26.2
- new net: R27.1, R28.2
Changed lines of the file:
@@
 	1    0    0    -1
 $EndComp
-Text GLabel 7950 2550 0    60   Input ~ 0
+Text GLabel 7900 2450 0    60   Input ~ 0
 OUT3
-Text GLabel 7950 900  0    60   Input ~ 0
+Text GLabel 7900 800  0    60   Input ~ 0
 OUT1
-Text GLabel 7950 1700 0    60   Input ~ 0
+Text GLabel 7900 1600 0    60   Input ~ 0
 OUT2
-Text GLabel 7950 3450 0    60   Input ~ 0
+Text GLabel 7900 3350 0    60   Input ~ 0
 OUT4
 Text GLabel 9400 2550 2    60   Input ~ 0
@@
 	10450 2150 10650 2150
 Wire Wire Line
-	7950 3450 8200 3450
-Wire Wire Line
-	7950 2550 8200 2550
-Wire Wire Line
-	7950 1700 8200 1700
-Wire Wire Line
-	7950 900  8200 900
-Wire Wire Line
 	10650 2250 10150 2250
 Wire Wire Line
@@
 Wire Wire Line
 	1350 4900 1450 4900
+$Comp
+L Device:R R21
+U 1 1 5DE92298
+P 8050 800
+F 0 "R21" V 8150 800 50  0000 C CNN
+F 1 "1.2k" V 8050 800 50  0000 C CNN
+F 2 "Resistor_SMD:R_0805_2012Metric_Pad1.15x1.40mm_HandSolder" V 7980 800 50  0001 C CNN
+F 3 "" H 8050 800 50  0000 C CNN
+	1    8050 800
+	0    1    1    0
+$EndComp
+$Comp
+L Device:R R22
+U 1 1 5DE9229F
+P 8050 1000
+F 0 "R22" V 7950 1000 50  0000 C CNN
+F 1 "1.2k" V 8050 1000 50  0000 C CNN
+F 2 "Resistor_SMD:R_0805_2012Metric_Pad1.15x1.40mm_HandSolder" V 7980 1000 50  0001 C CNN
+F 3 "" H 8050 1000 50  0000 C CNN
+	1    8050 1000
+	0    -1   -1   0
+$EndComp
+$Comp
+L power:GND #PWR0102
+U 1 1 5DE922A6
+P 7900 1000
+F 0 "#PWR0102" H 7900 750 50  0001 C CNN
+F 1 "GND" H 7750 1000 50  0000 C CNN
+F 2 "" H 7900 1000 50  0000 C CNN
+F 3 "" H 7900 1000 50  0000 C CNN
+	1    7900 1000
+	1    0    0    -1
+$EndComp
+Wire Wire Line
+	8200 800  8200 1000
+$Comp
+L Device:R R23
+U 1 1 5DE9BF84
+P 8050 1600
+F 0 "R23" V 8150 1600 50  0000 C CNN
+F 1 "1.2k" V 8050 1600 50  0000 C CNN
+F 2 "Resistor_SMD:R_0805_2012Metric_Pad1.15x1.40mm_HandSolder" V 7980 1600 50  0001 C CNN
+F 3 "" H 8050 1600 50  0000 C CNN
+	1    8050 1600
+	0    1    1    0
+$EndComp
+$Comp
+L Device:R R24
+U 1 1 5DE9BF8B
+P 8050 1800
+F 0 "R24" V 7950 1800 50  0000 C CNN
+F 1 "1.2k" V 8050 1800 50  0000 C CNN
+F 2 "Resistor_SMD:R_0805_2012Metric_Pad1.15x1.40mm_HandSolder" V 7980 1800 50  0001 C CNN
+F 3 "" H 8050 1800 50  0000 C CNN
+	1    8050 1800
+	0    -1   -1   0
+$EndComp
+$Comp
+L power:GND #PWR0103
+U 1 1 5DE9BF92
+P 7900 1800
+F 0 "#PWR0103" H 7900 1550 50  0001 C CNN
+F 1 "GND" H 7750 1750 50  0000 C CNN
+F 2 "" H 7900 1800 50  0000 C CNN
+F 3 "" H 7900 1800 50  0000 C CNN
+	1    7900 1800
+	1    0    0    -1
+$EndComp
+Wire Wire Line
+	8200 1600 8200 1800
+$Comp
+L Device:R R25
+U 1 1 5DEA5D08
+P 8050 2450
+F 0 "R25" V 8150 2450 50  0000 C CNN
+F 1 "1.2k" V 8050 2450 50  0000 C CNN
+F 2 "Resistor_SMD:R_0805_2012Metric_Pad1.15x1.40mm_HandSolder" V 7980 2450 50  0001 C CNN
+F 3 "" H 8050 2450 50  0000 C CNN
+	1    8050 2450
+	0    1    1    0
+$EndComp
+$Comp
+L Device:R R26
+U 1 1 5DEA5D0F
+P 8050 2650
+F 0 "R26" V 7950 2650 50  0000 C CNN
+F 1 "1.2k" V 8050 2650 50  0000 C CNN
+F 2 "Resistor_SMD:R_0805_2012Metric_Pad1.15x1.40mm_HandSolder" V 7980 2650 50  0001 C CNN
+F 3 "" H 8050 2650 50  0000 C CNN
+	1    8050 2650
+	0    -1   -1   0
+$EndComp
+$Comp
+L power:GND #PWR0104
+U 1 1 5DEA5D16
+P 7900 2650
+F 0 "#PWR0104" H 7900 2400 50  0001 C CNN
+F 1 "GND" H 7750 2600 50  0000 C CNN
+F 2 "" H 7900 2650 50  0000 C CNN
+F 3 "" H 7900 2650 50  0000 C CNN
+	1    7900 2650
+	1    0    0    -1
+$EndComp
+Wire Wire Line
+	8200 2450 8200 2650
+$Comp
+L Device:R R27
+U 1 1 5DEAF6B6
+P 8050 3350
+F 0 "R27" V 8150 3350 50  0000 C CNN
+F 1 "1.2k" V 8050 3350 50  0000 C CNN
+F 2 "Resistor_SMD:R_0805_2012Metric_Pad1.15x1.40mm_HandSolder" V 7980 3350 50  0001 C CNN
+F 3 "" H 8050 3350 50  0000 C CNN
+	1    8050 3350
+	0    1    1    0
+$EndComp
+$Comp
+L Device:R R28
+U 1 1 5DEAF6BD
+P 8050 3550
+F 0 "R28" V 7950 3550 50  0000 C CNN
+F 1 "1.2k" V 8050 3550 50  0000 C CNN
+F 2 "Resistor_SMD:R_0805_2012Metric_Pad1.15x1.40mm_HandSolder" V 7980 3550 50  0001 C CNN
+F 3 "" H 8050 3550 50  0000 C CNN
+	1    8050 3550
+	0    -1   -1   0
+$EndComp
+$Comp
+L power:GND #PWR0105
+U 1 1 5DEAF6C4
+P 7900 3550
+F 0 "#PWR0105" H 7900 3300 50  0001 C CNN
+F 1 "GND" H 7750 3500 50  0000 C CNN
+F 2 "" H 7900 3550 50  0000 C CNN
+F 3 "" H 7900 3550 50  0000 C CNN
+	1    7900 3550
+	1    0    0    -1
+$EndComp
+Wire Wire Line
+	8200 3350 8200 3550
 $EndSCHEMATC
