File: discrette_out/mosfet_out.sch (KiCad schematic (older format))
At the start: 5 parts

Commit message: Added some chematics
Parts:
- added R?: 6.3K, Resistor_SMD:R_0805_2012Metric_Pad1.15x1.40mm_HandSolder, symbol Device:R
Connections:
- net at Q?.1 (G), R?.2: now also R?.1; no longer U?.4
- net DOUT renamed DOUT_?
- net MCU_DOUT renamed MCU_DOUT_?
- new net: R?.2, U?.4
Other:
- moved on the sheet: D?, Q?, R?
Changed lines of the file:
@@
 L Device:D D?
 U 1 1 5EA2BF30
-P 5800 3350
-F 0 "D?" V 5754 3429 50  0000 L CNN
-F 1 "D" V 5845 3429 50  0000 L CNN
-F 2 "" H 5800 3350 50  0001 C CNN
-F 3 "~" H 5800 3350 50  0001 C CNN
-	1    5800 3350
+P 6000 3050
+F 0 "D?" V 5954 3129 50  0000 L CNN
+F 1 "D" V 6045 3129 50  0000 L CNN
+F 2 "" H 6000 3050 50  0001 C CNN
+F 3 "~" H 6000 3050 50  0001 C CNN
+	1    6000 3050
 	0    1    1    0
 $EndComp
-Text GLabel 5800 3900 2    50   Input ~ 0
-DOUT
-Text GLabel 5750 2850 2    50   Input ~ 0
+Text GLabel 6100 3600 2    50   Input ~ 0
+DOUT_?
+Text GLabel 6100 2550 2    50   Input ~ 0
 COMM_POW
 $Comp
 L Device:R R?
 U 1 1 5EA2C2AD
-P 5000 3100
-F 0 "R?" H 5070 3146 50  0000 L CNN
-F 1 "10K" H 5070 3055 50  0000 L CNN
-F 2 "Resistor_SMD:R_0805_2012Metric_Pad1.15x1.40mm_HandSolder" V 4930 3100 50  0001 C CNN
-F 3 "~" H 5000 3100 50  0001 C CNN
-	1    5000 3100
+P 5000 2750
+F 0 "R?" H 5070 2796 50  0000 L CNN
+F 1 "10K" H 5070 2705 50  0000 L CNN
+F 2 "Resistor_SMD:R_0805_2012Metric_Pad1.15x1.40mm_HandSolder" V 4930 2750 50  0001 C CNN
+F 3 "~" H 5000 2750 50  0001 C CNN
+	1    5000 2750
 	1    0    0    -1
 $EndComp
@@
 	4400 4200 4400 4350
 Text GLabel 3950 3500 0    50   Input ~ 0
-MCU_DOUT
+MCU_DOUT_?
 $Comp
 L Device:Q_PMOS_GDS Q?
 U 1 1 5EA2CA53
-P 5350 3350
-F 0 "Q?" H 5556 3396 50  0000 L CNN
-F 1 "AO3401A" H 5100 3200 50  0000 L CNN
-F 2 "" H 5550 3450 50  0001 C CNN
-F 3 "~" H 5350 3350 50  0001 C CNN
-	1    5350 3350
+P 5550 3050
+F 0 "Q?" H 5756 3096 50  0000 L CNN
+F 1 "AO3401A" H 5300 2900 50  0000 L CNN
+F 2 "" H 5750 3150 50  0001 C CNN
+F 3 "~" H 5550 3050 50  0001 C CNN
+	1    5550 3050
 	1    0    0    -1
 $EndComp
 Wire Wire Line
-	5000 3250 5000 3350
-Wire Wire Line
 	5000 4350 5000 3700
 Wire Wire Line
-	5000 2950 5000 2850
+	5650 2850 5650 2750
 Wire Wire Line
-	5150 3350 5000 3350
-Connection ~ 5000 3350
+	5650 3250 5650 3350
 Wire Wire Line
-	5000 3350 5000 3500
+	6000 3350 5650 3350
+Connection ~ 5650 3350
 Wire Wire Line
-	5450 3150 5450 3050
+	5650 3350 5650 3600
 Wire Wire Line
-	5450 2850 5000 2850
+	6000 2750 5650 2750
 Wire Wire Line
-	5750 2850 5450 2850
-Connection ~ 5450 2850
+	6000 3350 6000 3200
 Wire Wire Line
-	5450 3550 5450 3650
+	6000 2750 6000 2900
+$Comp
+L Device:R R?
+U 1 1 5EA2D5D5
+P 5000 3300
+F 0 "R?" H 5070 3346 50  0000 L CNN
+F 1 "6.3K" H 5070 3255 50  0000 L CNN
+F 2 "Resistor_SMD:R_0805_2012Metric_Pad1.15x1.40mm_HandSolder" V 4930 3300 50  0001 C CNN
+F 3 "~" H 5000 3300 50  0001 C CNN
+	1    5000 3300
+	1    0    0    -1
+$EndComp
 Wire Wire Line
-	5450 3900 5800 3900
+	5000 3500 5000 3450
 Wire Wire Line
-	5800 3650 5450 3650
-Connection ~ 5450 3650
+	5000 3150 5000 3050
 Wire Wire Line
-	5450 3650 5450 3900
+	5000 2600 5000 2550
 Wire Wire Line
-	5800 3050 5450 3050
-Connection ~ 5450 3050
+	5350 3050 5000 3050
+Connection ~ 5000 3050
 Wire Wire Line
-	5450 3050 5450 2850
+	5000 3050 5000 2900
 Wire Wire Line
-	5800 3650 5800 3500
+	6100 2550 5650 2550
 Wire Wire Line
-	5800 3050 5800 3200
+	5650 2750 5650 2550
+Connection ~ 5650 2750
+Connection ~ 5650 2550
+Wire Wire Line
+	5650 2550 5000 2550
+Wire Wire Line
+	6100 3600 5650 3600
 $EndSCHEMATC
